File: kicad/StepperDriver.kicad_pcb (KiCad board)
At the start: 2 copper layers, 0 parts

Commit message: Changed diode footprints
Parts:
- added C1: 100µF, Capacitor_THT:CP_Radial_D6.3mm_P2.50mm, F.Cu at (66.2, 44.5)
- added C10: 100nF, Capacitor_SMD:C_0805_2012Metric_Pad1.15x1.40mm_HandSolder, F.Cu at (57.8, 49.9)
- added C11: 100nF, Capacitor_SMD:C_0805_2012Metric_Pad1.15x1.40mm_HandSolder, F.Cu at (27.3, 58.4)
- added C12: 100nF, Capacitor_SMD:C_0805_2012Metric_Pad1.15x1.40mm_HandSolder, F.Cu at (32.0, 61.7)
- added C13: 1µF, Capacitor_SMD:C_0805_2012Metric_Pad1.15x1.40mm_HandSolder, F.Cu at (42.9, 51.7)
- added C14: 10nF, Capacitor_SMD:C_0805_2012Metric_Pad1.15x1.40mm_HandSolder, F.Cu at (76.3, 31.2)
- added C15: 10µF, Capacitor_SMD:C_0805_2012Metric_Pad1.15x1.40mm_HandSolder, F.Cu at (68.3, 39.0)
- added C16: 10µF, Capacitor_SMD:C_0805_2012Metric_Pad1.15x1.40mm_HandSolder, F.Cu at (27.3, 61.3)
- added C17: 1µF, Capacitor_SMD:C_0805_2012Metric_Pad1.15x1.40mm_HandSolder, F.Cu at (46.3, 62.1)
- added C18: 100µF, Capacitor_THT:CP_Radial_D6.3mm_P2.50mm, F.Cu at (88.7, 23.6)
- added C19: 1µF, Capacitor_SMD:C_0805_2012Metric_Pad1.15x1.40mm_HandSolder, F.Cu at (36.8, 61.7)
- added C2: 1000µF, Capacitor_THT:CP_Radial_D10.0mm_P5.00mm, F.Cu at (19.2, 50.4)
- added C20: 100µF, Capacitor_THT:CP_Radial_D6.3mm_P2.50mm, F.Cu at (58.2, 44.5)
- added C21: 100nF, Capacitor_SMD:C_0805_2012Metric_Pad1.15x1.40mm_HandSolder, F.Cu at (62.5, 49.9)
- added C22: 100nF, Capacitor_SMD:C_0805_2012Metric_Pad1.15x1.40mm_HandSolder, F.Cu at (41.5, 62.1)
- added C23: 10nF, Capacitor_SMD:C_0805_2012Metric_Pad1.15x1.40mm_HandSolder, F.Cu at (72.0, 49.9)
- added C24: 1µF, Capacitor_SMD:C_0805_2012Metric_Pad1.15x1.40mm_HandSolder, F.Cu at (68.9, 58.8)
- added C25: 100µF, Capacitor_THT:CP_Radial_D6.3mm_P2.50mm, F.Cu at (68.7, 33.6)
- added C26: 1µF, Capacitor_SMD:C_0805_2012Metric_Pad1.15x1.40mm_HandSolder, F.Cu at (76.8, 48.9)
- added C27: 100µF, Capacitor_THT:CP_Radial_D6.3mm_P2.50mm, F.Cu at (51.8, 58.1)
- added C28: 100nF, Capacitor_SMD:C_0805_2012Metric_Pad1.15x1.40mm_HandSolder, F.Cu at (64.1, 61.7)
- added C29: 100nF, Capacitor_SMD:C_0805_2012Metric_Pad1.15x1.40mm_HandSolder, F.Cu at (90.5, 34.9)
- added C3: 100µF, Capacitor_THT:CP_Radial_D6.3mm_P2.50mm, F.Cu at (80.7, 23.6)
- added C30: 100nF, Capacitor_SMD:C_0805_2012Metric_Pad1.15x1.40mm_HandSolder, F.Cu at (88.0, 37.9)
- added C4: 1000µF, Capacitor_THT:CP_Radial_D10.0mm_P5.00mm, F.Cu at (54.7, 19.0)
- added C5: 10µF, Capacitor_SMD:C_0805_2012Metric_Pad1.15x1.40mm_HandSolder, F.Cu at (81.0, 32.0)
- added C6: 1µF, Capacitor_SMD:C_0805_2012Metric_Pad1.15x1.40mm_HandSolder, F.Cu at (85.8, 29.0)
- added C7: 1µF, Capacitor_SMD:C_0805_2012Metric_Pad1.15x1.40mm_HandSolder, F.Cu at (81.0, 29.0)
- added C8: 4.7µF, Capacitor_SMD:C_0805_2012Metric_Pad1.15x1.40mm_HandSolder, F.Cu at (76.3, 37.1)
- added C9: 100nF, Capacitor_SMD:C_0805_2012Metric_Pad1.15x1.40mm_HandSolder, F.Cu at (76.3, 34.1)
- added D1: B540C, Diode_SMD:D_SMC_Handsoldering, F.Cu at (28.7, 33.0)
- added D2: B540C, Diode_SMD:D_SMC_Handsoldering, F.Cu at (43.5, 24.9)
- added D3: B540C, Diode_SMD:D_SMC_Handsoldering, F.Cu at (28.9, 17.1)
- added D4: B540C, Diode_SMD:D_SMC_Handsoldering, F.Cu at (13.8, 25.2)
- added D5: B540C, Diode_SMD:D_SMC_Handsoldering, F.Cu at (13.8, 33.0)
- added D6: B540C, Diode_SMD:D_SMC_Handsoldering, F.Cu at (28.7, 25.2)
- added D7: B540C, Diode_SMD:D_SMC_Handsoldering, F.Cu at (43.8, 17.1)
- added D8: B540C, Diode_SMD:D_SMC_Handsoldering, F.Cu at (13.8, 40.8)
- added D9: SMAJ16A, Diode_SMD:D_SMA_Handsoldering, F.Cu at (11.4, 59.1)
- added J1: Phase 1, footprints:20020327-C02xB0xLF, F.Cu at (51.2, 49.5)
- added J10: 2A, Jumper:SolderJumper-2_P1.3mm_Open_Pad1.0x1.5mm, F.Cu at (32.3, 75.2)
- added J11: 3A, Jumper:SolderJumper-2_P1.3mm_Open_Pad1.0x1.5mm, F.Cu at (36.7, 72.3)
- added J12: 3A, Jumper:SolderJumper-2_P1.3mm_Open_Pad1.0x1.5mm, F.Cu at (32.3, 71.7)
- added J13: 4A, Jumper:SolderJumper-2_P1.3mm_Open_Pad1.0x1.5mm, F.Cu at (31.5, 82.3)
- added J14: 4A, Jumper:SolderJumper-2_P1.3mm_Open_Pad1.0x1.5mm, F.Cu at (36.7, 75.8)
- added J15: 5A, Jumper:SolderJumper-2_P1.3mm_Open_Pad1.0x1.5mm, F.Cu at (31.9, 78.8)
- added J16: 5A, Jumper:SolderJumper-2_P1.3mm_Open_Pad1.0x1.5mm, F.Cu at (27.2, 81.1)
- added J2: BOOT0, Connector_PinHeader_2.54mm:PinHeader_1x02_P2.54mm_Vertical, F.Cu at (23.6, 39.2)
- added J3: Phase 2, footprints:20020327-C02xB0xLF, F.Cu at (61.6, 29.5)
- added J4: Power In, footprints:20020327-C02xB0xLF, F.Cu at (73.7, 17.9)
- added J5: USART, Connector_PinHeader_2.54mm:PinHeader_1x04_P2.54mm_Vertical, F.Cu at (13.4, 47.0)
- added J6: Control IO, Connector_PinHeader_2.54mm:PinHeader_1x04_P2.54mm_Vertical, F.Cu at (8.71, 47.0)
- added J7: 1A, Jumper:SolderJumper-2_P1.3mm_Open_Pad1.0x1.5mm, F.Cu at (22.8, 80.5)
- added J8: 1A, Jumper:SolderJumper-2_P1.3mm_Open_Pad1.0x1.5mm, F.Cu at (37.1, 68.7)
- added J9: 2A, Jumper:SolderJumper-2_P1.3mm_Open_Pad1.0x1.5mm, F.Cu at (27.6, 77.6)
- added NT1: NT, NetTie:NetTie-2_SMD_Pad0.5mm, F.Cu at (11.0, 62.5)
- added NT2: NT, NetTie:NetTie-2_SMD_Pad0.5mm, F.Cu at (7.91, 62.5)
- added R1: 10k, Resistor_SMD:R_0805_2012Metric_Pad1.15x1.40mm_HandSolder, F.Cu at (64.1, 58.8)
- added R10: 1R, Resistor_SMD:R_0805_2012Metric_Pad1.15x1.40mm_HandSolder, F.Cu at (59.4, 58.8)
- added R11: 1R, Resistor_SMD:R_0805_2012Metric_Pad1.15x1.40mm_HandSolder, F.Cu at (85.8, 32.0)
- added R12: 1R, Resistor_SMD:R_0805_2012Metric_Pad1.15x1.40mm_HandSolder, F.Cu at (59.4, 52.9)
- added R13: 1R, Resistor_SMD:R_0805_2012Metric_Pad1.15x1.40mm_HandSolder, F.Cu at (78.5, 40.0)
- added R14: 1k, Resistor_SMD:R_0805_2012Metric_Pad1.15x1.40mm_HandSolder, F.Cu at (64.1, 55.8)
- added R15: 1R, Resistor_SMD:R_0805_2012Metric_Pad1.15x1.40mm_HandSolder, F.Cu at (73.7, 46.0)
- added R16: 1R, Resistor_SMD:R_0805_2012Metric_Pad1.15x1.40mm_HandSolder, F.Cu at (68.9, 52.9)
- added R17: 1R, Resistor_SMD:R_0805_2012Metric_Pad1.15x1.40mm_HandSolder, F.Cu at (78.5, 43.0)
- added R18: 1R, Resistor_SMD:R_0805_2012Metric_Pad1.15x1.40mm_HandSolder, F.Cu at (85.8, 34.9)
- added R19: 1R, Resistor_SMD:R_0805_2012Metric_Pad1.15x1.40mm_HandSolder, F.Cu at (59.4, 61.7)
- added R2: 1R, Resistor_SMD:R_0805_2012Metric_Pad1.15x1.40mm_HandSolder, F.Cu at (90.5, 29.0)
- added R20: 1R, Resistor_SMD:R_0805_2012Metric_Pad1.15x1.40mm_HandSolder, F.Cu at (73.7, 43.0)
- added R21: 1R, Resistor_SMD:R_0805_2012Metric_Pad1.15x1.40mm_HandSolder, F.Cu at (78.5, 46.0)
- added R22: 1R, Resistor_SMD:R_0805_2012Metric_Pad1.15x1.40mm_HandSolder, F.Cu at (68.9, 55.8)
- added R23: 100k, Resistor_SMD:R_0805_2012Metric_Pad1.15x1.40mm_HandSolder, F.Cu at (83.2, 40.8)
- added R24: 100k, Resistor_SMD:R_0805_2012Metric_Pad1.15x1.40mm_HandSolder, F.Cu at (83.2, 37.9)
- added R25: 1k, Resistor_SMD:R_0805_2012Metric_Pad1.15x1.40mm_HandSolder, F.Cu at (13.5, 80.2)
- added R26: 1k, Resistor_SMD:R_0805_2012Metric_Pad1.15x1.40mm_HandSolder, F.Cu at (23.0, 71.4)
- added R27: 1k, Resistor_SMD:R_0805_2012Metric_Pad1.15x1.40mm_HandSolder, F.Cu at (27.8, 68.4)
- added R28: 1k, Resistor_SMD:R_0805_2012Metric_Pad1.15x1.40mm_HandSolder, F.Cu at (18.3, 83.2)
- added R29: 1k, Resistor_SMD:R_0805_2012Metric_Pad1.15x1.40mm_HandSolder, F.Cu at (18.3, 74.3)
- added R3: 1R, Resistor_SMD:R_0805_2012Metric_Pad1.15x1.40mm_HandSolder, F.Cu at (64.1, 52.9)
- added R30: 1k, Resistor_SMD:R_0805_2012Metric_Pad1.15x1.40mm_HandSolder, F.Cu at (13.5, 77.3)
- added R31: 1k, Resistor_SMD:R_0805_2012Metric_Pad1.15x1.40mm_HandSolder, F.Cu at (23.0, 68.4)
- added R32: 1k, Resistor_SMD:R_0805_2012Metric_Pad1.15x1.40mm_HandSolder, F.Cu at (8.76, 80.2)
- added R33: 1k, Resistor_SMD:R_0805_2012Metric_Pad1.15x1.40mm_HandSolder, F.Cu at (18.3, 71.4)
- added R34: 1k, Resistor_SMD:R_0805_2012Metric_Pad1.15x1.40mm_HandSolder, F.Cu at (13.5, 74.3)
- added R35: 7k15, Resistor_SMD:R_0805_2012Metric_Pad1.15x1.40mm_HandSolder, F.Cu at (8.76, 77.3)
- added R36: 7k15, Resistor_SMD:R_0805_2012Metric_Pad1.15x1.40mm_HandSolder, F.Cu at (18.3, 68.4)
- added R37: 10k, Resistor_SMD:R_0805_2012Metric_Pad1.15x1.40mm_HandSolder, F.Cu at (13.5, 71.4)
- added R38: 1k, Resistor_SMD:R_0805_2012Metric_Pad1.15x1.40mm_HandSolder, F.Cu at (8.76, 74.3)
- added R39: 10k, Resistor_SMD:R_0805_2012Metric_Pad1.15x1.40mm_HandSolder, F.Cu at (13.5, 68.4)
- added R4: 1R, Resistor_SMD:R_0805_2012Metric_Pad1.15x1.40mm_HandSolder, F.Cu at (59.4, 55.8)
- added R40: 1k, Resistor_SMD:R_0805_2012Metric_Pad1.15x1.40mm_HandSolder, F.Cu at (8.76, 71.4)
- added R41: 10k, Resistor_SMD:R_0805_2012Metric_Pad1.15x1.40mm_HandSolder, F.Cu at (8.76, 83.2)
- added R42: 10k, Resistor_SMD:R_0805_2012Metric_Pad1.15x1.40mm_HandSolder, F.Cu at (18.3, 77.3)
- added R43: 10k, Resistor_SMD:R_0805_2012Metric_Pad1.15x1.40mm_HandSolder, F.Cu at (8.76, 68.4)
- added R44: 10k, Resistor_SMD:R_0805_2012Metric_Pad1.15x1.40mm_HandSolder, F.Cu at (23.0, 74.3)
- added R45: 10k, Resistor_SMD:R_0805_2012Metric_Pad1.15x1.40mm_HandSolder, F.Cu at (13.5, 83.2)
- added R46: 10k, Resistor_SMD:R_0805_2012Metric_Pad1.15x1.40mm_HandSolder, F.Cu at (27.8, 71.4)
- added R47: 10k, Resistor_SMD:R_0805_2012Metric_Pad1.15x1.40mm_HandSolder, F.Cu at (18.3, 80.2)
- added R48: 10k, Resistor_SMD:R_0805_2012Metric_Pad1.15x1.40mm_HandSolder, F.Cu at (32.5, 68.4)
- added R49: 10k, Resistor_SMD:R_0805_2012Metric_Pad1.15x1.40mm_HandSolder, F.Cu at (23.0, 77.3)
- added R5: 1R, Resistor_SMD:R_0805_2012Metric_Pad1.15x1.40mm_HandSolder, F.Cu at (67.3, 49.9)
- added R50: 10k, Resistor_SMD:R_0805_2012Metric_Pad1.15x1.40mm_HandSolder, F.Cu at (27.8, 74.3)
- added R6: 1R, Resistor_SMD:R_0805_2012Metric_Pad1.15x1.40mm_HandSolder, F.Cu at (90.5, 32.0)
- added R7: 1R, Resistor_SMD:R_0805_2012Metric_Pad1.15x1.40mm_HandSolder, F.Cu at (81.0, 34.9)
- added R8: 1R, Resistor_SMD:R_0805_2012Metric_Pad1.15x1.40mm_HandSolder, F.Cu at (73.7, 40.0)
- added R9: 1R, Resistor_SMD:R_0805_2012Metric_Pad1.15x1.40mm_HandSolder, F.Cu at (73.6, 52.9)
- added SW1: Reset, footprints:LL3301NF065QG, F.Cu at (13.9, 17.3)
- added U1: AP7370, Package_TO_SOT_SMD:SOT-23, F.Cu at (83.1, 44.6)
- added U10: FAN3278, Package_SO:SOIC-8_3.9x4.9mm_P1.27mm, F.Cu at (70.0, 26.5)
- added U11: FAN3278, Package_SO:SOIC-8_3.9x4.9mm_P1.27mm, F.Cu at (90.5, 16.5)
- added U12: MCP6L02, Package_SO:SOIC-8_3.9x4.9mm_P1.27mm, F.Cu at (20.7, 59.4)
- added U13: MCP6L02, Package_SO:SOIC-8_3.9x4.9mm_P1.27mm, F.Cu at (61.7, 37.4)
- added U14: FAN3278, Package_SO:SOIC-8_3.9x4.9mm_P1.27mm, F.Cu at (82.1, 16.5)
- added U15: FAN3278, Package_SO:SOIC-8_3.9x4.9mm_P1.27mm, F.Cu at (44.8, 57.4)
- added U16: STM32F303K6Tx, Package_QFP:LQFP-32_7x7mm_P0.8mm, F.Cu at (41.8, 34.5)
- added U2: FDS4435BZ, footprints:SO-8_MOSFET, F.Cu at (66.3, 18.3)
- added U3: FDS4435BZ, footprints:SO-8_MOSFET, F.Cu at (30.8, 51.9)
- added U4: FDS4435BZ, footprints:SO-8_MOSFET, F.Cu at (37.3, 45.2)
- added U5: FDS4435BZ, footprints:SO-8_MOSFET, F.Cu at (50.8, 39.8)
- added U6: DMG4496SSS, footprints:SO-8_MOSFET, F.Cu at (37.3, 55.2)
- added U7: DMG4496SSS, footprints:SO-8_MOSFET, F.Cu at (54.2, 29.8)
- added U8: DMG4496SSS, footprints:SO-8_MOSFET, F.Cu at (30.8, 41.9)
- added U9: DMG4496SSS, footprints:SO-8_MOSFET, F.Cu at (43.8, 45.2)
Other:
- rule pad_to_mask_clearance: 0.051 -> 0.001
- rule solder_mask_min_width: 0.25 -> 0.2

Commit message: Some kind of beginning of layout
Parts:
- removed the U13 at (61.7, 37.4)
- D1, D2, D3, D4, D5, D6, D7, D8: footprint Diode_SMD:D_SMC_Handsoldering -> Diode_SMD:D_SMC
- D9: footprint Diode_SMD:D_SMA_Handsoldering -> Diode_SMD:D_SMA
- U2, U3, U4, U5, U6, U7, U8, U9: footprint footprints:SO-8_MOSFET -> Package_SO:SOIC-8_3.9x4.9mm_P1.27mm
- moved U15 131.7 mm to (172.2, 52.8)
- moved NT1 116.2 mm to (120.9, 24.8)
- moved NT2 116.2 mm to (117.8, 24.8)
- moved U12 110.6 mm to (110.2, 124.4)
- moved J7 108.5 mm to (130.5, 93.6)
- moved J9 108.5 mm to (135.3, 90.7)
- moved R25 108.5 mm to (121.2, 93.3)
- moved R28 108.5 mm to (126.0, 96.3)
- moved R29 108.5 mm to (126.0, 87.4)
- moved R30 108.5 mm to (121.2, 90.4)
- moved R32 108.5 mm to (116.5, 93.3)
- moved R33 108.5 mm to (126.0, 84.5)
- moved R34 108.5 mm to (121.2, 87.4)
- moved R35 108.5 mm to (116.5, 90.4)
- moved R36 108.5 mm to (126.0, 81.5)
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- renumbered U14 to U13, U15 to U14, U16 to U15
Connections:
- U10 pad 2: /P1_4 -> /P1_2
- U10 pad 7: /P1_FET4 -> /P1_FET2
- U11 pad 2: /P1_2 -> /P1_4
- U11 pad 7: /P1_FET2 -> /P1_FET4
- U12 pad 5: (no net) -> /P2_SENSE
- U12 pad 6: (no net) -> /CurrentSelection/P2_GAIN
- U12 pad 7: (no net) -> /IP2
- U13 pad 2: /P2_4 -> /P2_2
- U13 pad 7: /P2_FET4 -> /P2_FET2
- U14 pad 2: /P2_2 -> /P2_4
- U14 pad 7: /P2_FET2 -> /P2_FET4
- U2 pad 1: /P1_FET1 -> VDD
- U2 pad 2: /P1.1 -> VDD
- U3 pad 1: /P1_FET3 -> VDD
- U3 pad 2: /P1.2 -> VDD
- U4 pad 1: /P2_FET1 -> VDD
- U4 pad 2: /P2.1 -> VDD
- U5 pad 1: /P2_FET3 -> VDD
- U5 pad 2: /P2.2 -> VDD
- U6 pad 1: /P1_FET2 -> /P1_SENSE
- U6 pad 2: /P1.1 -> /P1_SENSE
- U7 pad 1: /P1_FET4 -> /P1_SENSE
- U7 pad 2: /P1.2 -> /P1_SENSE
- U8 pad 1: /P2_FET2 -> /P2_SENSE
- U8 pad 2: /P2.1 -> /P2_SENSE
- U9 pad 1: /P2_FET4 -> /P2_SENSE
- U9 pad 2: /P2.2 -> /P2_SENSE

Commit message: Some other form of layout
Parts:
- removed the C20 at (129.5, 44.5)
- removed the C21 at (131.8, 52.2)
- removed the C26 at (146.1, 51.2)
- removed C27: 100µF, Capacitor_THT:CP_Radial_D6.3mm_P2.50mm
- removed C28, C29: 100nF, Capacitor_SMD:C_0805_2012Metric_Pad1.15x1.40mm_HandSolder
- added C19: 1µF, Capacitor_SMD:C_0805_2012Metric_Pad1.15x1.40mm_HandSolder, F.Cu at (10.5, 54.5)
- added C23: 10µF, Capacitor_SMD:C_0805_2012Metric_Pad1.15x1.40mm_HandSolder, F.Cu at (57.0, 54.5)
- C17: value 1µF -> 10µF
- C18: value 100µF -> 10µF; footprint Capacitor_THT:CP_Radial_D6.3mm_P2.50mm -> Capacitor_SMD:C_0805_2012Metric_Pad1.15x1.40mm_HandSolder
- C22: value 100nF -> 10µF
- C25: value 100µF -> 1µF; footprint Capacitor_THT:CP_Radial_D6.3mm_P2.50mm -> Capacitor_SMD:C_0805_2012Metric_Pad1.15x1.40mm_HandSolder
- D1, D2, D3, D4, D5, D6, D7, D8: moved to B.Cu
- moved R2 135.9 mm to (15.0, 68.0)
- moved R6 135.7 mm to (15.0, 70.0)
- moved R11 129.1 mm to (21.0, 72.0)
- moved C18 124.2 mm to (23.5, 54.5), turned to 90 degrees
- moved R7 124.0 mm to (21.0, 70.0)
- moved R15 122.4 mm to (15.0, 74.0)
- moved R16 118.7 mm to (21.0, 74.0)
- moved R20 116.6 mm to (21.0, 76.0)
- moved R19 114.3 mm to (15.0, 76.0)
- moved R10 114.2 mm to (15.0, 72.0)
- moved R3 113.1 mm to (21.0, 68.0)
- moved C17 103.9 mm to (12.5, 54.5), turned to 90 degrees
- moved R18 95.7 mm to (54.5, 74.0)
- moved C24 94.4 mm to (44.0, 54.5), turned to 90 degrees
- moved R17 93.8 mm to (48.5, 74.0)
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- renumbered C19 to C20, C23 to C21, C30 to C26
Connections:
- U15 pad 16: GND -> GNDD
- U15 pad 32: GND -> GNDD
Routing:
- net VDD: track 0.00 -> 68.1 mm
- net GND: track 0.00 -> 33.0 mm
- net /P2_FET2: track 0.00 -> 24.5 mm
- net /P1_FET2: track 0.00 -> 24.5 mm
- net /P2_FET4: track 0.00 -> 21.6 mm, vias 0 -> 2
- net /P1_FET4: track 0.00 -> 21.6 mm, vias 0 -> 2
- net /P2_FET1: track 0.00 -> 15.6 mm
- net /P1_FET1: track 0.00 -> 15.6 mm
- net /P2_FET3: track 0.00 -> 14.5 mm
- net /P1_FET3: track 0.00 -> 14.5 mm
- added copper zone on B.Cu, net (none)
- added copper zone on F.Cu, net (none)
- added copper zone on B.Cu, net /P1.1
- added copper zone on F.Cu, net /P1.1
- added copper zone on B.Cu, net /P1.2
- added copper zone on F.Cu, net /P1.2
- added copper zone on F.Cu, net /P1_SENSE

Commit message: Fixed zone net
Routing:
- added copper zone on B.Cu, net /P2.1
- added copper zone on F.Cu, net /P2.1
- added copper zone on B.Cu, net /P2.2
- added copper zone on F.Cu, net /P2.2
- added copper zone on F.Cu, net /P2_SENSE
- removed copper zone on B.Cu, net (none)
- removed copper zone on F.Cu, net (none)
Changed lines of the file:
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@@
     (user_trace_width 0.25)
     (trace_clearance 0.2)
-    (zone_clearance 0.508)
+    (zone_clearance 0.2)
     (zone_45_only no)
     (trace_min 0.1)
@@
     )
   )
-  (zone (net 0) (net_name "") (layer F.Cu) (hatch edge 0.508)
+  (zone (net 30) (net_name /P2_SENSE) (layer F.Cu) (hatch edge 0.508)
     (connect_pads yes (clearance 0.2))
     (min_thickness 0.15)
@@
     )
   )
-  (zone (net 0) (net_name "") (layer F.Cu) (hatch edge 0.508)
+  (zone (net 10) (net_name /P2.2) (layer F.Cu) (hatch edge 0.508)
     (connect_pads yes (clearance 0.2))
     (min_thickness 0.15)
@@
     )
   )
-  (zone (net 0) (net_name "") (layer B.Cu) (hatch edge 0.508)
+  (zone (net 10) (net_name /P2.2) (layer B.Cu) (hatch edge 0.508)
     (connect_pads yes (clearance 0.508))
     (min_thickness 0.254)
@@
     )
   )
-  (zone (net 0) (net_name "") (layer B.Cu) (hatch edge 0.508)
+  (zone (net 9) (net_name /P2.1) (layer B.Cu) (hatch edge 0.508)
     (connect_pads yes (clearance 0.508))
     (min_thickness 0.254)
@@
     )
   )
-  (zone (net 0) (net_name "") (layer F.Cu) (hatch edge 0.508)
+  (zone (net 9) (net_name /P2.1) (layer F.Cu) (hatch edge 0.508)
     (connect_pads yes (clearance 0.2))
     (min_thickness 0.15)
